File: AMS GIGA Display CANBus/AMS GIGA Display CANBus.kicad_pcb (KiCad board)
At the start: 2 copper layers, 101.6 x 53.3 mm, 27 parts, among them J1 Power, J2 PWM, J3 Analog, J4 PWM, J5 Analog, J6 Communication, J7 Digital, J8 Power_And_CAN, J9 Conn_01x02, Q1 IRF9Z34NPBF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

Commit message: added some silkscreen labeling that i forgot to add before fab oh well.
Other:
- board text added: "1 Amp"
- board text added: "120 Ohm Termination Resistor Jumper"
- board text added: "12V"
- board text added: "AMS GIGA Display V 1.0 Rev A"
- board text added: "CH"
- board text added: "CL"
- board text added: "GND"
Changed lines of the file:
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@@
 		(tags "TVS Diode (Uni-directional)")
 		(property "Reference" "D1"
-			(at 3.075 0 0)
+			(at 3.075 0.215 0)
 			(layer "F.SilkS")
 			(effects
@@
 		(tags "MOSFET (N-Channel)")
 		(property "Reference" "Q1"
-			(at 6.58 3 0)
+			(at 9.58 -1.5 0)
 			(layer "F.SilkS")
 			(effects
@@
 		(layer "Edge.Cuts")
 	)
+	(gr_text "CL"
+		(at 105 78.5 0)
+		(layer "F.SilkS")
+		(effects
+			(font
+				(size 1 1)
+				(thickness 0.15)
+			)
+			(justify left bottom)
+		)
+	)
+	(gr_text "12V"
+		(at 105 71 0)
+		(layer "F.SilkS")
+		(effects
+			(font
+				(size 1 1)
+				(thickness 0.15)
+			)
+			(justify left bottom)
+		)
+	)
+	(gr_text "GND"
+		(at 105 73.5 0)
+		(layer "F.SilkS")
+		(effects
+			(font
+				(size 1 1)
+				(thickness 0.15)
+			)
+			(justify left bottom)
+		)
+	)
+	(gr_text "1 Amp"
+		(at 141 63.5 0)
+		(layer "F.SilkS")
+		(effects
+			(font
+				(size 1 1)
+				(thickness 0.15)
+			)
+			(justify left bottom)
+		)
+	)
+	(gr_text "CH"
+		(at 105 76 0)
+		(layer "F.SilkS")
+		(effects
+			(font
+				(size 1 1)
+				(thickness 0.15)
+			)
+			(justify left bottom)
+		)
+	)
+	(gr_text "AMS GIGA Display\nV 1.0 Rev A"
+		(at 170.5 65 0)
+		(layer "F.SilkS")
+		(effects
+			(font
+				(size 1 1)
+				(thickness 0.15)
+			)
+			(justify left bottom)
+		)
+	)
+	(gr_text "120 Ohm Termination\nResistor Jumper"
+		(at 120.5 69.5 0)
+		(layer "F.SilkS")
+		(effects
+			(font
+				(size 1 1)
+				(thickness 0.15)
+			)
+			(justify left bottom)
+		)
+	)
 	(gr_text "ICSP"
